Commit message: sunny

File: catkin_ws/src/30-localization-and-planning/duckietown_description/urdf/macros.urdf.xacro (robot description, xacro)
@@ -3,4 +3,10 @@
     <xacro:property name="pi" value="3.14159265359" />
     <xacro:property name="tile_thickness" value="0.01" />
+	<physics type='ode'>
+      <max_step_size>0.001</max_step_size>
+      <real_time_factor>1</real_time_factor>
+      <real_time_update_rate>1000</real_time_update_rate>
+      <gravity>0 0 -9.8</gravity>
+    </physics>
     <!-- Defines a tile link and joint-->
     <xacro:macro name="tile" params="x y type:=empty rotation:=0 visible:=true">
@@ -10,9 +16,38 @@
                     <origin xyz="${tile_width/2} ${tile_width/2} ${-tile_thickness/2}" rpy="0 0 ${rotation * pi/180}"/>
                     <geometry>
-                        <mesh filename="package://duckietown_description/urdf/meshes/${type}.dae" />
+                        <mesh filename="package://duckietown_description/urdf/meshes/${type}.dae" scale="1.02 1.02 1.02"/>
                     </geometry>
                 </visual>
+		<inertial>
+    			<origin xyz="${tile_width/2} ${tile_width/2} ${-tile_thickness/2}" rpy="0 0 0"/>
+    			<mass value="100"/>
+     			<inertia  ixx="0" ixy = "0" ixz = "0"
+    			iyy="0" iyz = "0"
+    			izz="0"/>
+  		</inertial>
+	    <collision>
+    		<origin xyz="${tile_width/2} ${tile_width/2} ${-tile_thickness/2}" rpy="0 0 0"/>
+    		<geometry>
+      			 <box size="${tile_width} ${tile_width} ${tile_thickness}"/>
+    		</geometry>
+		<surface>
+            <friction>
+              <ode>
+                <mu>100</mu>
+                <mu2>50</mu2>
+              </ode>
+            </friction>
+            <bounce/>
+            <contact>
+              <ode/>
+            </contact>
+          </surface>
+          <max_contacts>10</max_contacts>
+  		</collision>
             </xacro:if>
         </link>
+	<gazebo>
+    <static>true</static>
+	</gazebo>
         <joint name="world_to_tile_${x}_${y}" type="fixed">
             <parent link="world" />
@@ -21,4 +56,5 @@
         </joint>
     </xacro:macro>
+<!-- *************************************************************-->
     <!-- Defines an april tag link and joint-->
     <xacro:macro name="tag" params="id x y pos rotation">

Commit message: lane following

File: catkin_ws/src/30-localization-and-planning/duckietown_description/urdf/macros.urdf.xacro (robot description, xacro)
@@ -16,5 +16,5 @@
                     <origin xyz="${tile_width/2} ${tile_width/2} ${-tile_thickness/2}" rpy="0 0 ${rotation * pi/180}"/>
                     <geometry>
-                        <mesh filename="package://duckietown_description/urdf/meshes/${type}.dae" scale="1.02 1.02 1.02"/>
+                        <mesh filename="package://duckietown_description/urdf/meshes/${type}.dae" scale="1.0084 1.0084 1.0084"/>
                     </geometry>
                 </visual>
